Commit message: Rename packages

File: pincher_arm_description/urdf/arm_hardware.xacro (robot description, xacro)
@@ -33,5 +33,5 @@
         <origin xyz="-0.028 -0.0493 0.014" rpy="0.0 0.0 -${pi/2}"/>
         <geometry>
-          <mesh filename="package://phantomx_pincher_arm_description/meshes/mount.stl" scale="${M_SCALE} ${M_SCALE} ${M_SCALE}"/>
+          <mesh filename="package://pincher_arm_description/meshes/mount.stl" scale="${M_SCALE} ${M_SCALE} ${M_SCALE}"/>
         </geometry>
         <material name="${color}"/>
@@ -61,5 +61,5 @@
         <origin xyz="0 0 0" rpy="0 0 0"/>
         <geometry>
-          <mesh filename="package://phantomx_pincher_arm_description/meshes/ax12_box.stl" scale="${M_SCALE} ${M_SCALE} ${M_SCALE}"/>
+          <mesh filename="package://pincher_arm_description/meshes/ax12_box.stl" scale="${M_SCALE} ${M_SCALE} ${M_SCALE}"/>
         </geometry>
         <material name="Black"/>
@@ -89,5 +89,5 @@
         <origin xyz="0 0 0" rpy="0 0 0"/>
         <geometry>
-          <mesh filename="package://phantomx_pincher_arm_description/meshes/F10.stl" scale="${M_SCALE} ${M_SCALE} ${M_SCALE}"/>
+          <mesh filename="package://pincher_arm_description/meshes/F10.stl" scale="${M_SCALE} ${M_SCALE} ${M_SCALE}"/>
         </geometry>
         <material name="${color}"/>
@@ -117,5 +117,5 @@
         <origin xyz="0 0 0" rpy="0 0 0"/>
         <geometry>
-          <mesh filename="package://phantomx_pincher_arm_description/meshes/F3.stl" scale="${M_SCALE} ${M_SCALE} ${M_SCALE}"/>
+          <mesh filename="package://pincher_arm_description/meshes/F3.stl" scale="${M_SCALE} ${M_SCALE} ${M_SCALE}"/>
         </geometry>
         <material name="${color}"/>
@@ -148,5 +148,5 @@
         <origin xyz="0 0 0" rpy="0 0 0"/>
         <geometry>
-          <mesh filename="package://phantomx_pincher_arm_description/meshes/F3.stl" scale="${M_SCALE} ${M_SCALE} ${M_SCALE}"/>
+          <mesh filename="package://pincher_arm_description/meshes/F3.stl" scale="${M_SCALE} ${M_SCALE} ${M_SCALE}"/>
         </geometry>
         <material name="${color}"/>
@@ -179,5 +179,5 @@
         <origin xyz="0 0 0" rpy="0 0 0"/>
         <geometry>
-          <mesh filename="package://phantomx_pincher_arm_description/meshes/F2.stl" scale="${M_SCALE} ${M_SCALE} ${M_SCALE}"/>
+          <mesh filename="package://pincher_arm_description/meshes/F2.stl" scale="${M_SCALE} ${M_SCALE} ${M_SCALE}"/>
         </geometry>
         <material name="${color}"/>
@@ -210,5 +210,5 @@
         <origin xyz="0 0 0" rpy="0 0 0"/>
         <geometry>
-          <mesh filename="package://phantomx_pincher_arm_description/meshes/F4.stl" scale="${M_SCALE} ${M_SCALE} ${M_SCALE}"/>
+          <mesh filename="package://pincher_arm_description/meshes/F4.stl" scale="${M_SCALE} ${M_SCALE} ${M_SCALE}"/>
         </geometry>
         <material name="${color}"/>
@@ -260,5 +260,5 @@
         <xacro:insert_block name="origin"/>
         <geometry>
-          <mesh filename="package://phantomx_pincher_arm_description/meshes/pincher_finger.stl" scale=".01 .01 .01"/>
+          <mesh filename="package://pincher_arm_description/meshes/pincher_finger.stl" scale=".01 .01 .01"/>
         </geometry>
         <material name="${color}"/>

File: pincher_arm_description/urdf/pincher_arm.urdf.xacro (robot description, xacro)
@@ -1,5 +1,5 @@
 <?xml version="1.0"?>
 <robot name="pincher_arm" xmlns:xacro="http://ros.org/wiki/xacro">
-  <xacro:include filename="$(find phantomx_pincher_arm_description)/urdf/pincher_arm.xacro"/>
+  <xacro:include filename="$(find pincher_arm_description)/urdf/pincher_arm.xacro"/>
   <link name="base_link"/>
   <xacro:pincher_arm parent="base_link">

File: pincher_arm_description/urdf/pincher_arm.xacro (robot description, xacro)
@@ -2,5 +2,5 @@
 <!-- PhantomX Pincher arm description -->
 <robot xmlns:xacro="http://ros.org/wiki/xacro">
-  <xacro:include filename="$(find phantomx_pincher_arm_description)/urdf/arm_hardware.xacro"/>
+  <xacro:include filename="$(find pincher_arm_description)/urdf/arm_hardware.xacro"/>
   <material name="White">
     <color rgba="0.87 0.90 0.87 1.0"/>

Commit message: Modify finger origins

File: pincher_arm_description/urdf/arm_hardware.xacro (robot description, xacro)
@@ -254,5 +254,5 @@
     </gazebo>
   </xacro:macro>
-  <xacro:macro name="pincher_gripper" params="name color *origin">
+  <xacro:macro name="pincher_finger" params="name color *origin">
     <link name="${name}_link">
       <xacro:box_inertia length="0.036" width="0.028" height="0.004" mass="0.00001"/>

File: pincher_arm_description/urdf/pincher_arm.xacro (robot description, xacro)
@@ -111,7 +111,7 @@
     </joint>
     <!-- Finger 1 -->
-    <xacro:pincher_gripper name="gripper_finger1" color="${color}" >
-      <origin xyz="0 0.01 0" rpy="${pi/2} 0 ${pi/2}"/>
-    </xacro:pincher_gripper>
+    <xacro:pincher_finger name="gripper_finger1" color="${color}" >
+      <origin xyz="0 0.0115 0" rpy="${pi/2} 0 ${pi/2}"/>
+    </xacro:pincher_finger>
     <joint name="gripper_finger1_joint" type="prismatic">
       <origin xyz="0.019 0 0" rpy="0 0 0"/>
@@ -122,7 +122,7 @@
     </joint>
     <!-- Finger 2 -->
-    <xacro:pincher_gripper name="gripper_finger2" color="${color}" >
-      <origin xyz="0 0.01 0" rpy="${pi/2} 0 ${pi/2}"/>
-    </xacro:pincher_gripper>
+    <xacro:pincher_finger name="gripper_finger2" color="${color}" >
+      <origin xyz="0 0.0115 0" rpy="${pi/2} 0 ${pi/2}"/>
+    </xacro:pincher_finger>
     <joint name="gripper_finger2_joint" type="prismatic">
       <origin xyz="0.019 0 0" rpy="${pi} 0 0"/>
