Commit message: Change structure of gripper URDF

File: pincher_arm_description/urdf/pincher_arm.xacro (robot description, xacro)
@@ -27,4 +27,6 @@
       wrist_llimit:=-1.72
       wrist_ulimit:=1.68
+      gripper_llimit:=-2.6
+      gripper_ulimit:=0.0
       *origin">
     <link name="arm_base_link"/>
@@ -100,32 +102,40 @@
       <origin xyz="0  ${AX12_WIDTH/2} 0" rpy="${pi} 0 ${pi/2}"/>
     </xacro:gripper_finger_base>
+    <link name="gripper_active_link"/>
+    <joint name="gripper_joint" type="revolute">
+      <origin xyz="0 0 0" rpy="0 0 0"/>
+      <axis xyz="1 0 0"/>
+      <limit effort="30" velocity="${joints_vlimit}" lower="${gripper_llimit}" upper="${gripper_ulimit}"/>
+      <parent link="gripper_finger_base_link"/>
+      <child link="gripper_active_link"/>
+    </joint>
     <!-- Finger 1 -->
-    <joint name="gripper_joint" type="prismatic">
+    <xacro:pincher_gripper name="gripper_finger1" color="${color}" >
+      <origin xyz="0 0.01 0" rpy="${pi/2} 0 ${pi/2}"/>
+    </xacro:pincher_gripper>
+    <joint name="gripper_finger1_joint" type="prismatic">
       <origin xyz="0.019 0 0" rpy="0 0 0"/>
       <axis xyz="0 1 0"/>
       <limit effort="30" velocity="0.05" lower="0.001" upper="0.0175"/>
       <parent link="gripper_finger_base_link"/>
-      <child link="gripper_active_link"/>
+      <child link="gripper_finger1_link"/>
     </joint>
-    <xacro:pincher_gripper name="gripper_active" color="${color}" >
+    <!-- Finger 2 -->
+    <xacro:pincher_gripper name="gripper_finger2" color="${color}" >
       <origin xyz="0 0.01 0" rpy="${pi/2} 0 ${pi/2}"/>
     </xacro:pincher_gripper>
-    <!-- Finger 2 -->
-    <joint name="gripper2_joint" type="prismatic">
+    <joint name="gripper_finger2_joint" type="prismatic">
       <origin xyz="0.019 0 0" rpy="${pi} 0 0"/>
       <axis xyz="0 1 0"/>
       <limit effort="30" velocity="0.05" lower="0.001" upper="0.0175"/>
       <parent link="gripper_finger_base_link"/>
-      <child link="gripper_active2_link"/>
-      <mimic joint="gripper_joint"/>
+      <child link="gripper_finger2_link"/>
+      <mimic joint="gripper_finger1_joint"/>
     </joint>
-    <xacro:pincher_gripper name="gripper_active2" color="${color}" >
-      <origin xyz="0 0.01 0" rpy="${pi/2} 0 ${pi/2}"/>
-    </xacro:pincher_gripper>
     <!-- fake gripper joint -->
     <link name="gripper_fake_link"/>
     <joint name="gripper_fake_joint" type="revolute">
-      <origin xyz="0 0 0.085" rpy="0 -1.57 0"/>
-      <parent link="arm_wrist_flex_link"/>
+      <origin xyz="0 0 0.02" rpy="0 0 0"/>
+      <parent link="gripper_finger_base_link"/>
       <child link="gripper_fake_link"/>
       <limit effort="30" velocity="1" lower="-3.14" upper="3.14"/>

Commit message: Update upper limits for fingers

File: pincher_arm_description/urdf/pincher_arm.xacro (robot description, xacro)
@@ -117,5 +117,5 @@
       <origin xyz="0.019 0 0" rpy="0 0 0"/>
       <axis xyz="0 1 0"/>
-      <limit effort="30" velocity="0.05" lower="0.001" upper="0.0175"/>
+      <limit effort="30" velocity="0.05" lower="0.001" upper="0.0158"/>
       <parent link="gripper_finger_base_link"/>
       <child link="gripper_finger1_link"/>
@@ -128,5 +128,5 @@
       <origin xyz="0.019 0 0" rpy="${pi} 0 0"/>
       <axis xyz="0 1 0"/>
-      <limit effort="30" velocity="0.05" lower="0.001" upper="0.0175"/>
+      <limit effort="30" velocity="0.05" lower="0.001" upper="0.0158"/>
       <parent link="gripper_finger_base_link"/>
       <child link="gripper_finger2_link"/>

Commit message: Remove mimic tag to resolve problems with moveit parallel gripper controller

File: pincher_arm_description/urdf/pincher_arm.xacro (robot description, xacro)
@@ -117,5 +117,5 @@
       <origin xyz="0.019 0 0" rpy="0 0 0"/>
       <axis xyz="0 1 0"/>
-      <limit effort="30" velocity="0.05" lower="0.001" upper="0.0158"/>
+      <limit effort="30" velocity="0.01" lower="0.001" upper="0.0158"/>
       <parent link="gripper_finger_base_link"/>
       <child link="gripper_finger1_link"/>
@@ -128,8 +128,8 @@
       <origin xyz="0.019 0 0" rpy="${pi} 0 0"/>
       <axis xyz="0 1 0"/>
-      <limit effort="30" velocity="0.05" lower="0.001" upper="0.0158"/>
+      <limit effort="30" velocity="0.01" lower="0.001" upper="0.0158"/>
       <parent link="gripper_finger_base_link"/>
       <child link="gripper_finger2_link"/>
-      <mimic joint="gripper_finger1_joint"/>
+      <!-- <mimic joint="gripper_finger1_joint"/> -->
     </joint>
     <!-- fake gripper joint -->

Commit message: Fix gripper_fake_link location

File: pincher_arm_description/urdf/pincher_arm.xacro (robot description, xacro)
@@ -136,5 +136,5 @@
     <link name="gripper_fake_link"/>
     <joint name="gripper_fake_joint" type="revolute">
-      <origin xyz="0 0 0.02" rpy="0 0 0"/>
+      <origin xyz="0.02 0 0" rpy="0 0 0"/>
       <parent link="gripper_finger_base_link"/>
       <child link="gripper_fake_link"/>

Commit message: Don't add base_link to URDF

File: pincher_arm_description/urdf/pincher_arm.xacro (robot description, xacro)
@@ -16,5 +16,4 @@
   </material>
   <xacro:macro name="pincher_arm" params="
-      parent:=base_link
       color:=Gray
       joints_vlimit:=1.571
@@ -28,12 +27,6 @@
       wrist_ulimit:=1.79
       gripper_llimit:=-2.6
-      gripper_ulimit:=0.0
-      *origin">
+      gripper_ulimit:=0.0">
     <link name="arm_base_link"/>
-    <joint name="arm_base_joint" type="fixed">
-      <xacro:insert_block name="origin"/>
-      <parent link="${parent}"/>
-      <child link="arm_base_link"/>
-    </joint>
     <!-- shoulder pan joint -->
     <xacro:dynamixel_AX12_fixed parent="arm_base_link" name="arm_shoulder_pan_servo">
